File: hardware/bldc_motor_controller_schematic.kicad_pcb (KiCad board)
At the start: 2 copper layers, 115 x 89 mm, 12 parts, among them J1 Conn_02x19_Odd_Even, J10 J_BARREL_JACK1, J2 Conn_02x19_Odd_Even, J3 J_AS5600, J4 J_INA226, J5 J_SSD1306, J6 J_HM10, J7 J_DRV8313_CTRL

Commit message: feat(hardware): route all nets on the carrier PCB
- Route the 12 V and VM motor supply path through the INA226 at 1.0 mm

- Add a GND pour across the bottom layer

- Route the UART, I2C, 3V3, 5V, PWM, EN, and nFT nets, splitting I2C and 3V3 across both layers to avoid crossings

- Narrow the Logic net class to 0.3 mm so traces fit between the Morpho header pads

- Remove a 3V3 track stub so DRC passes with no errors or warnings
Routing:
- net +3V3: track 0.00 -> 211.6 mm
- net /nFT: track 0.00 -> 111.1 mm
- net /SDA: track 0.00 -> 94.9 mm
- net /EN: track 0.00 -> 92.2 mm
- net /SCL: track 0.00 -> 89.7 mm, vias 0 -> 1
- net /VM: track 0.00 -> 52.2 mm
- net +5V: track 0.00 -> 39.7 mm
- net /PWM_IN1: track 0.00 -> 37.4 mm
- net /PWM_IN3: track 0.00 -> 35.0 mm
- net /UART_RX: track 0.00 -> 24.1 mm
- net /PWM_IN2: track 0.00 -> 23.4 mm
- net +12V: track 0.00 -> 21.8 mm
- net /UART_TX: track 0.00 -> 15.9 mm
- added copper zone on B.Cu, net GND

Commit message: feat(hardware): finalize carrier PCB for fabrication
- Rotate the SSD1306 connector so the display reads upright, and reroute its 3V3, SCL, and SDA traces

- Add silkscreen pin labels for the power, encoder, HM-10, OLED, and INA226 connectors

- Add board name, version, and author to the silkscreen
Parts:
- moved J5 12.3 mm to (178.9, 67.8), turned to 90 degrees
Routing:
- net /SDA: track 94.9 -> 126.7 mm
- net /SCL: track 89.7 -> 117.1 mm
- net +3V3: track 211.6 -> 233.3 mm
Other:
- board text added: "12V"
- board text added: "3V3"
- board text added: "BLDC CARRIER v1.0"
- board text added: "CN10"
- board text added: "CN7"
- board text added: "GND"
- board text added: "IN+"
- board text added: "RXD"
- board text added: "S. CHIARAMONTE 2026"
- board text added: "SCL"
- board text added: "SDA"
- board text added: "TXD"
- board text added: "VCC"
